File: Awesome-Shield-0.50/Awesome-Shield-0.5.sch (EAGLE design)
At the start: 37 parts, among them SW1 SPST_TACT-EVQQ2, U1 LIGHTSENSORTEMT6000

Commit message: adjusted sch to make refdes more visible
Parts:
- renumbered S2 to SW2
Other:
- moved on the sheet: JP1, JP2, JP3, JP4, LED1, R1, R10, R2, R5, R8, R9

Commit message: added refdes labels for THT parts to silkscreen, image export broken - images out of date
Parts:
- renumbered J3 to J1, J4 to J2
Changed lines of the file:
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@@
 <part name="R10" library="rcl" deviceset="R-EU_" device="R0603" value="130 Ohm"/>
 <part name="R11" library="rcl" deviceset="R-EU_" device="R0603" value="10K"/>
-<part name="J3" library="Seeed-OPL-Connector" deviceset="GROVE-CONNECTOR-SMD(4+2P-2.0)" device=""/>
-<part name="J4" library="Seeed-OPL-Connector" deviceset="GROVE-CONNECTOR-SMD(4+2P-2.0)" device=""/>
+<part name="J1" library="Seeed-OPL-Connector" deviceset="GROVE-CONNECTOR-SMD(4+2P-2.0)" device=""/>
+<part name="J2" library="Seeed-OPL-Connector" deviceset="GROVE-CONNECTOR-SMD(4+2P-2.0)" device=""/>
 <part name="FID1" library="SparkFun-Aesthetics" deviceset="FIDUCIAL" device="1X2"/>
 <part name="FID2" library="SparkFun-Aesthetics" deviceset="FIDUCIAL" device="1X2"/>
@@
 <instance part="R10" gate="G$1" x="254" y="127"/>
 <instance part="R11" gate="G$1" x="193.04" y="190.5" rot="R90"/>
-<instance part="J3" gate="G$1" x="180.34" y="57.15"/>
-<instance part="J4" gate="G$1" x="337.82" y="64.77"/>
+<instance part="J1" gate="G$1" x="180.34" y="57.15"/>
+<instance part="J2" gate="G$1" x="337.82" y="64.77"/>
 <instance part="FID1" gate="G$1" x="15.24" y="15.24"/>
 <instance part="FID2" gate="G$1" x="20.32" y="15.24"/>
@@
 <pinref part="GND6" gate="1" pin="GND"/>
 <wire x1="167.64" y1="53.34" x2="175.26" y2="53.34" width="0.1524" layer="91"/>
-<pinref part="J3" gate="G$1" pin="4"/>
+<pinref part="J1" gate="G$1" pin="4"/>
 </segment>
 <segment>
@@
 <pinref part="GND7" gate="1" pin="GND"/>
 <wire x1="320.04" y1="58.42" x2="320.04" y2="55.88" width="0.1524" layer="91"/>
-<pinref part="J4" gate="G$1" pin="4"/>
+<pinref part="J2" gate="G$1" pin="4"/>
 </segment>
 <segment>
@@
 <wire x1="180.34" y1="48.26" x2="180.34" y2="45.72" width="0.1524" layer="91"/>
 <junction x="180.34" y="48.26"/>
-<pinref part="J3" gate="G$1" pin="SS1"/>
-<pinref part="J3" gate="G$1" pin="SS2"/>
+<pinref part="J1" gate="G$1" pin="SS1"/>
+<pinref part="J1" gate="G$1" pin="SS2"/>
 </segment>
 <segment>
@@
 <wire x1="337.82" y1="55.88" x2="337.82" y2="53.34" width="0.1524" layer="91"/>
 <junction x="337.82" y="55.88"/>
-<pinref part="J4" gate="G$1" pin="SS1"/>
-<pinref part="J4" gate="G$1" pin="SS2"/>
+<pinref part="J2" gate="G$1" pin="SS1"/>
+<pinref part="J2" gate="G$1" pin="SS2"/>
 </segment>
 <segment>
@@
 <pinref part="P+1" gate="1" pin="+5V"/>
 <wire x1="175.26" y1="55.88" x2="167.64" y2="55.88" width="0.1524" layer="91"/>
-<pinref part="J3" gate="G$1" pin="3"/>
+<pinref part="J1" gate="G$1" pin="3"/>
 </segment>
 <segment>
@@
 <pinref part="P+2" gate="1" pin="+5V"/>
 <wire x1="320.04" y1="66.04" x2="320.04" y2="68.58" width="0.1524" layer="91"/>
-<pinref part="J4" gate="G$1" pin="3"/>
+<pinref part="J2" gate="G$1" pin="3"/>
 </segment>
 <segment>
@@
 <wire x1="327.66" y1="78.74" x2="317.5" y2="88.9" width="0.1524" layer="91"/>
 <wire x1="317.5" y1="88.9" x2="309.88" y2="88.9" width="0.1524" layer="91"/>
-<pinref part="J4" gate="G$1" pin="1"/>
+<pinref part="J2" gate="G$1" pin="1"/>
 </segment>
 <segment>
@@
 <pinref part="SJ2" gate="G$1" pin="1"/>
 <label x="170.18" y="68.58" size="1.778" layer="95"/>
-<pinref part="J3" gate="G$1" pin="1"/>
+<pinref part="J1" gate="G$1" pin="1"/>
 <label x="208.28" y="104.14" size="1.778" layer="95"/>
 </segment>
@@
 <pinref part="SJ1" gate="G$1" pin="1"/>
 <label x="162.56" y="68.58" size="1.778" layer="95"/>
-<pinref part="J3" gate="G$1" pin="2"/>
+<pinref part="J1" gate="G$1" pin="2"/>
 <label x="210.82" y="111.76" size="1.778" layer="95"/>
 </segment>
@@
 <wire x1="322.58" y1="81.28" x2="309.88" y2="81.28" width="0.1524" layer="91"/>
 <label x="309.88" y="81.28" size="1.778" layer="95"/>
-<pinref part="J4" gate="G$1" pin="2"/>
-</segment>
-<segment>
+<pinref part="J2" gate="G$1" pin="2"/>
+</segment>
+<segment>
