File: Awesome-Shield-0.60/Awesome-Shield-0.6.brd (EAGLE design)
At the start: 51 x 55 mm, 22 parts, among them J1 PORT1, J2 PORT2, J3 PORT3, SW1 SPST_TACT-EVQQ2, SW2 DPDT, U1 LIGHTSENSORTEMT6000

Commit message: changed fiducials to Watterott standard 0.7mm
Parts:
- removed FID1, FID3, FID4: FIDUCIAL1X2, SparkFun-Aesthetics:FIDUCIAL-1X2
- added X1, X2: PASSER-07, we-symbol:PASSER_07MM
Changed lines of the file:
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@@
 <attribute name="VALUE" x="5.207" y="20.955" size="0.889" layer="27" font="vector" ratio="11" rot="R90"/>
 </element>
-<element name="FID1" library="SparkFun-Aesthetics" package="FIDUCIAL-1X2" value="FIDUCIAL1X2" x="47.498" y="48.26"/>
-<element name="FID3" library="SparkFun-Aesthetics" package="FIDUCIAL-1X2" value="FIDUCIAL1X2" x="47.498" y="5.08"/>
-<element name="FID4" library="SparkFun-Aesthetics" package="FIDUCIAL-1X2" value="FIDUCIAL1X2" x="1.27" y="48.26"/>
 <element name="U1" library="SparkFun-Sensors" package="TEMT6000-SEN" value="LIGHTSENSORTEMT6000" x="21.59" y="13.335" smashed="yes" rot="R270"/>
 <element name="JP4" library="adafruit" package="1X10-BIG" value="PINHD-1X10" x="13.97" y="50.8" smashed="yes" rot="R180"/>
@@
 <element name="U$1" library="buzzer-loudity-bzel-t68-0808" package="SMT-68" value="LOUDITY-BZEL-T680808" x="38.735" y="43.18" smashed="yes" rot="R90"/>
 <element name="R2" library="we-rcl" package="C1206" value="330R" x="12.065" y="45.72"/>
+<element name="X1" library="we-symbol" package="PASSER_07MM" value="PASSER-07" x="1.27" y="48.26"/>
+<element name="X2" library="we-symbol" package="PASSER_07MM" value="PASSER-07" x="47.625" y="5.08"/>
 </elements>
 <signals>
