File: Awesome-Shield-1.0.brd (EAGLE design)
At the start: 51 x 55 mm, 24 parts, among them J1 PORT1, J2 PORT2, J3 PORT3, SW1 SPST_TACT-EVQQ2, SW2 DPDT, U1 LIGHTSENSORTEMT6000, X1 PASSER-07, X2 PASSER-07

Commit message: updated Gerbers - :shipit:
Parts:
- R1: value TBD -> 91R 1%
Changed lines of the file:
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@@
 </element>
 <element name="C1" library="rcl" package="C0603" value="100nF" x="22.86" y="38.1" smashed="yes"/>
-<element name="R1" library="rcl" package="R1206" value="TBD" x="31.115" y="46.99" smashed="yes" rot="R180"/>
+<element name="R1" library="rcl" package="R1206" value="91R 1%" x="31.115" y="46.99" smashed="yes" rot="R180"/>
 <element name="U$1" library="buzzer-loudity-bzel-t68-0808" package="SMT-68" value="LOUDITY-BZEL-T680808" x="38.735" y="43.18" smashed="yes" rot="R90"/>
 <element name="R2" library="we-rcl" package="C1206" value="330R" x="14.605" y="45.72" smashed="yes">
