File: Awesome-Shield-1.0.sch (EAGLE design)
At the start: 24 parts, among them J1 PORT1, J2 PORT2, J3 PORT3, SW1 SPST_TACT-EVQQ2, SW2 DPDT, U1 LIGHTSENSORTEMT6000, X1 PASSER-07, X2 PASSER-07

Commit message: updated Gerbers - :shipit:
Parts:
- R1: value TBD -> 91R 1%
Changed lines of the file:
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@@
 <part name="C1" library="rcl" deviceset="C-EU" device="C0603" value="100nF"/>
 <part name="GND13" library="supply1" deviceset="GND" device=""/>
-<part name="R1" library="rcl" deviceset="R-EU_" device="R1206" value="TBD"/>
+<part name="R1" library="rcl" deviceset="R-EU_" device="R1206" value="91R 1%"/>
 <part name="U$1" library="buzzer-loudity-bzel-t68-0808" deviceset="LOUDITY-BZEL-T68" device="0808"/>
 <part name="R2" library="we-rcl" deviceset="RESISTOR" device="-1206" value="330R"/>
